File: Back_PCB.kicad_sch (KiCad schematic)
At the start: 50 parts, among them J4 VDRIVE_OUT, J5 NIXIE_1_2_OUT, J6 NIXIE_3_4_OUT, J7 mini-DS-3231, J8 Flash, P1 USB_C_Plug, Q1 Q_NPN_BCE, Q2 Q_NPN_BCE, SW4 Boot, SW5 Rst, SW6 Volume_down, SW7 Volume_up, U5 ESP32-WROOM-32, U6 74HC164D,653, U7 DFPlayer_mini

Commit message: Final version without panelization.
Connections:
- net +3.3V is gone; now on net +3.3VP: J7.1 (Pin_1), R23.1, R24.1
- net +3.3VP: now also J4.4 (Pin_4), U5.2 (3V3); no longer J4.3 (Pin_3)
- net +5VP: now also J4.3 (Pin_3); no longer J4.4 (Pin_4)
- net ENC_CLK_: now also U5.37 (IO23); no longer U5.26 (IO4)
- net GND: now also C6.2, C7.2
- net N1_A: now also U5.9 (IO33); no longer U5.10 (IO25)
- net N1_B: now also U5.11 (IO26); no longer U5.36 (IO22)
- net N1_C: now also U5.12 (IO27); no longer U5.33 (IO21)
- net N1_D: now also U5.10 (IO25); no longer U5.37 (IO23)
- net N2_A: now also U5.26 (IO4); no longer U5.9 (IO33)
- net N2_B: now also U5.31 (IO19); no longer U5.12 (IO27)
- net N2_C: now also U5.33 (IO21); no longer U5.11 (IO26)
- net N2_D: now also U5.29 (IO5); no longer U5.8 (IO32)
- net NX_SHDN: now also U5.8 (IO32); no longer U5.29 (IO5)
- net SHIFT_DSA: now also U5.36 (IO22); no longer U5.31 (IO19)
Other:
- moved on the sheet: C6, C7
