File: power.kicad_sch (KiCad schematic)
At the start: 17 parts, among them SW8 PWR_SW, U10 DD05CVSA, U11 Nixie-PSU, U12 Mini360, U8 AMS1117-5.0, U9 DD04CPMA

Commit message: Final version without panelization.
Parts:
- U10: value DD05CVSA -> DD04CVSA; footprint Retro_clock:DD05CVSA -> Retro_clock:DD04CVSA
Other:
- note added: "DD05CVSA changed to 10 watt DD04CVSA"
- note added: "Ich = 1A Iout = 0.8A Idis = 3.5A Vin = 4.5-6.5V"
- note removed: "Ich = 1A Iout = 1.2A Idis = 2A Vin = 4.5-8V"
Changed lines of the file:
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@@
+    (effects (font (size 1.27 1.27)) (justify left bottom))
+  )
+  (text "DD05CVSA changed to 10 watt DD04CVSA" (at 40.5638 52.7558 0)
     (effects (font (size 1.27 1.27)) (justify left bottom))
   )
@@
     (effects (font (size 1.27 1.27)) (justify left bottom))
   )
-  (text "Ich = 1A\nIout = 1.2A\nIdis = 2A\nVin = 4.5-8V" (at 48.7302 27.212 0)
+  (text "Ich = 1A\nIout = 0.8A\nIdis = 3.5A\nVin = 4.5-6.5V" (at 48.7302 27.212 0)
     (effects (font (size 1.27 1.27)) (justify left bottom))
   )
@@
     (in_bom yes) (on_board yes) (fields_autoplaced)
     (property "Reference" "U10" (id 0) (at 54.5846 29.3202 0))
-    (property "Value" "DD05CVSA" (id 1) (at 54.5846 31.8571 0))
-    (property "Footprint" "Retro_clock:DD05CVSA" (id 2) (at 61.3156 42.2402 0)
+    (property "Value" "DD04CVSA" (id 1) (at 54.5846 31.8571 0))
+    (property "Footprint" "Retro_clock:DD04CVSA" (id 2) (at 61.3156 42.2402 0)
       (effects (font (size 1.27 1.27)) hide)
     )
