File: Retro_clock.kicad_pcb (KiCad board)
At the start: 2 copper layers, 140 x 76.9 mm, 34 parts, among them J1 Conn_01x08_Female, J2 Conn_01x08_Female, J3 Conn_01x10_Female, SW1 Rotary_Encoder_Switch, SW2 KLS7-TS6601-13.0-180, SW3 KLS7-TS6601-13.0-180, U1 K155ID1, U2 K155ID1, U3 K155ID1, U4 K155ID1

Commit message: Finished first pcb, 2nd schematics and footprints.
Parts:
- removed G***: LOGO, NadSilk:brain_logo
- added BT1: 18560, Retro_clock:BAT_BH-18650-PC, B.Cu at (141.5, 137.2)
- added C10: Reserved_p, Capacitor_SMD:C_0603_1608Metric_Pad1.08x0.95mm_HandSolder, F.Cu at (252.0, 165.6)
- added C11: 0.1uF, Capacitor_SMD:C_0603_1608Metric_Pad1.08x0.95mm_HandSolder, F.Cu at (246.7, 173.2)
- added C12: Reserv, Capacitor_SMD:C_0603_1608Metric_Pad1.08x0.95mm_HandSolder, F.Cu at (252.0, 168.1)
- added C13: 10uF, Capacitor_SMD:C_0603_1608Metric_Pad1.08x0.95mm_HandSolder, F.Cu at (208.0, 78.1)
- added C14: 22uF, Capacitor_Tantalum_SMD:CP_EIA-3216-10_Kemet-I_Pad1.58x1.35mm_HandSolder, F.Cu at (208.9, 72.3)
- added C15: 10uF, Capacitor_SMD:C_0603_1608Metric_Pad1.08x0.95mm_HandSolder, F.Cu at (212.8, 75.1)
- added C16: 0.1uF, Capacitor_SMD:C_0603_1608Metric_Pad1.08x0.95mm_HandSolder, F.Cu at (248.2, 198.1)
- added C17: 10uF, Capacitor_SMD:C_0805_2012Metric_Pad1.18x1.45mm_HandSolder, F.Cu at (208.2, 75.3)
- added C18: 10uF, Capacitor_SMD:C_0603_1608Metric_Pad1.08x0.95mm_HandSolder, F.Cu at (226.6, 71.9)
- added C19: Reserv, Capacitor_SMD:C_0603_1608Metric_Pad1.08x0.95mm_HandSolder, F.Cu at (229.7, 194.4)
- added C20: 10uF, Capacitor_SMD:C_0603_1608Metric_Pad1.08x0.95mm_HandSolder, F.Cu at (214.1, 71.9)
- added C21: 0.1uF, Capacitor_SMD:C_0603_1608Metric_Pad1.08x0.95mm_HandSolder, F.Cu at (248.2, 200.6)
- added C6: 10uF, Capacitor_SMD:C_0603_1608Metric_Pad1.08x0.95mm_HandSolder, F.Cu at (218.4, 184.7)
- added C7: 0.1uF, Capacitor_SMD:C_0603_1608Metric_Pad1.08x0.95mm_HandSolder, F.Cu at (247.7, 170.7)
- added C8: 1uF, Capacitor_SMD:C_0603_1608Metric_Pad1.08x0.95mm_HandSolder, F.Cu at (247.7, 165.6)
- added C9: 1uF, Capacitor_SMD:C_0603_1608Metric_Pad1.08x0.95mm_HandSolder, F.Cu at (246.7, 175.7)
- added D1: ESDA5V3L, Package_TO_SOT_SMD:SOT-23, F.Cu at (210.0, 126.0)
- added F1: F2.5A, Fuse:Fuse_1206_3216Metric_Pad1.42x1.75mm_HandSolder, F.Cu at (289.8, 94.5)
- added F2: F40mA, Fuse:Fuse_1206_3216Metric_Pad1.42x1.75mm_HandSolder, F.Cu at (210.5, 117.0)
- added H5: MountingHole, MountingHole:MountingHole_2.5mm_Pad_Via, F.Cu at (53.5, 129.8)
- added H6: MountingHole, MountingHole:MountingHole_2.5mm_Pad_Via, F.Cu at (53.5, 199.6)
- added H7: MountingHole, MountingHole:MountingHole_2.5mm_Pad_Via, F.Cu at (186.1, 199.6)
- added H8: MountingHole, MountingHole:MountingHole_2.5mm_Pad_Via, F.Cu at (186.1, 129.8)
- added J4: VDRIVE_OUT, Connector_PinSocket_2.54mm:PinSocket_1x10_P2.54mm_Vertical, F.Cu at (106.9, 198.5)
- added J5: NIXIE_1_2_OUT, Connector_PinSocket_2.54mm:PinSocket_1x08_P2.54mm_Vertical, F.Cu at (94.0, 181.6)
- added J6: NIXIE_3_4_OUT, Connector_PinSocket_2.54mm:PinSocket_1x08_P2.54mm_Vertical, F.Cu at (145.4, 181.0)
- added J7: mini-DS-3231, Retro_clock:DS3231-Mini, F.Cu at (283.6, 182.4)
- added J8: Flash, Connector_PinHeader_2.54mm:PinHeader_1x05_P2.54mm_Vertical, F.Cu at (225.2, 190.9)
- added LS1: Speaker, Retro_clock:Speaker_conn, F.Cu at (319.2, 150.4)
- added P1: USB_C_Plug, Retro_clock:usb_c_receptable_hro_type-c-31-m-17, B.Cu at (70.7, 130.4)
- added Q1: Q_NPN_BCE, Package_TO_SOT_SMD:SOT-23_Handsoldering, F.Cu at (230.7, 190.9)
- added Q2: Q_NPN_BCE, Package_TO_SOT_SMD:SOT-23_Handsoldering, F.Cu at (237.2, 190.9)
- added R10: 10k, Resistor_SMD:R_0603_1608Metric_Pad0.98x0.95mm_HandSolder, F.Cu at (214.1, 184.7)
- added R11: 10k, Resistor_SMD:R_0603_1608Metric_Pad0.98x0.95mm_HandSolder, F.Cu at (242.1, 162.9)
- added R12: 10k, Resistor_SMD:R_0603_1608Metric_Pad0.98x0.95mm_HandSolder, F.Cu at (242.3, 173.2)
- added R13: 10k, Resistor_SMD:R_0603_1608Metric_Pad0.98x0.95mm_HandSolder, F.Cu at (205.4, 184.7)
- added R14: 250, Resistor_SMD:R_0603_1608Metric_Pad0.98x0.95mm_HandSolder, F.Cu at (256.4, 165.6)
- added R15: 250, Resistor_SMD:R_0603_1608Metric_Pad0.98x0.95mm_HandSolder, F.Cu at (242.3, 178.2)
- added R16: R, Resistor_SMD:R_0603_1608Metric_Pad0.98x0.95mm_HandSolder, F.Cu at (242.3, 175.7)
- added R17: R, Resistor_SMD:R_0603_1608Metric_Pad0.98x0.95mm_HandSolder, F.Cu at (209.8, 184.7)
- added R18: R, Resistor_SMD:R_0603_1608Metric_Pad0.98x0.95mm_HandSolder, F.Cu at (222.8, 184.7)
- added R19: R, Resistor_SMD:R_0603_1608Metric_Pad0.98x0.95mm_HandSolder, F.Cu at (237.8, 162.9)
- added R20: R, Resistor_SMD:R_0603_1608Metric_Pad0.98x0.95mm_HandSolder, F.Cu at (247.7, 168.1)
- added R21: R, Resistor_SMD:R_0603_1608Metric_Pad0.98x0.95mm_HandSolder, F.Cu at (262.2, 158.4)
- added R22: 10k, Resistor_SMD:R_0603_1608Metric_Pad0.98x0.95mm_HandSolder, F.Cu at (258.1, 189.9)
- added R23: 4.7k, Resistor_SMD:R_0603_1608Metric_Pad0.98x0.95mm_HandSolder, F.Cu at (229.7, 196.9)
- added R24: 4.7k, Resistor_SMD:R_0603_1608Metric_Pad0.98x0.95mm_HandSolder, F.Cu at (234.0, 194.4)
- added R25: 5.1k, Resistor_SMD:R_0603_1608Metric_Pad0.98x0.95mm_HandSolder, F.Cu at (201.6, 222.8)
- added R26: 5.1k, Resistor_SMD:R_0603_1608Metric_Pad0.98x0.95mm_HandSolder, F.Cu at (201.6, 220.3)
- added R27: 10k, Resistor_SMD:R_0603_1608Metric_Pad0.98x0.95mm_HandSolder, F.Cu at (197.2, 220.3)
- added R28: 10k, Resistor_SMD:R_0603_1608Metric_Pad0.98x0.95mm_HandSolder, F.Cu at (197.2, 222.8)
- added R29: 10k, Resistor_SMD:R_0603_1608Metric_Pad0.98x0.95mm_HandSolder, F.Cu at (240.1, 133.8)
- added R9: 10k, Resistor_SMD:R_0603_1608Metric_Pad0.98x0.95mm_HandSolder, F.Cu at (252.0, 170.7)
- added SW4: Boot, Retro_clock:SW_TS-1187A-B-A-B, F.Cu at (265.2, 153.3)
- added SW5: Rst, Retro_clock:SW_TS-1187A-B-A-B, F.Cu at (230.8, 165.4)
- added SW6: Volume_down, Retro_clock:KLS7-TS6601-13.0-180, F.Cu at (240.7, 168.2)
- added SW7: Volume_up, Retro_clock:KLS7-TS6601-13.0-180, F.Cu at (230.8, 172.9)
- added SW8: PWR_SW, Retro_clock:PWR_SWITCH, F.Cu at (26.7, 148.4)
- added U10: DD05CVSA, Retro_clock:DD05CVSA, B.Cu at (80.3, 143.9)
- added U11: Nixie-PSU, Retro_clock:Nixie-PSU, B.Cu at (117.8, 175.9)
- added U12: Mini360, Retro_clock:Mini360_step-down, F.Cu at (25.2, 182.7)
- added U5: ESP32-WROOM-32, Retro_clock:MODULE_ESP32-WROOM-32, F.Cu at (176.2, 167.4)
- added U6: 74HC164D,653, Retro_clock:SOIC127P600X175-14N, F.Cu at (106.3, 220.2)
- added U7: DFPlayer_mini, Retro_clock:MODULE_DFR0299, F.Cu at (165.4, 223.2)
- added U8: AMS1117-5.0, Package_TO_SOT_SMD:SOT-223-3_TabPin2, F.Cu at (11.2, 168.7)
- added U9: DD04CPMA, Retro_clock:DD04CPMA, B.Cu at (96.6, 131.8)
- added mouse-bite-1mm-slot: VAL**, Panelization:mouse-bite-1mm-slot, F.Cu at (190.0, 142.0)
- C2: footprint Capacitor_Tantalum_SMD:CP_EIA-7361-38_AVX-V_Pad2.18x3.30mm_HandSolder -> Capacitor_Tantalum_SMD:CP_EIA-3216-10_Kemet-I_Pad1.58x1.35mm_HandSolder
- SW2: value KLS7-TS6601-13.0-180 -> Enter
- SW3: value KLS7-TS6601-13.0-180 -> Cancel
- moved C3 4.23 mm to (119.8, 105.0)
- moved C2 2.30 mm to (116.7, 105.5)
Connections:
- net CLK renamed ENC_CLK
- net DATA renamed ENC_DATA
- J3 pad 3: unconnected-(J3-Pad3) -> +3.3V
- R5 pad 1: +5V -> +3.3V
- R6 pad 1: +5V -> +3.3V
Routing:
- net +3.3V: track 0.00 -> 22.5 mm, vias 0 -> 1
- net +5V: track 177.1 -> 166.4 mm
- net Earth: track 43.8 -> 38.6 mm, vias 8 -> 7
- added copper zone on B.Cu, net GND
Other:
- board size 140 x 76.9 mm -> 143.3 x 164.2 mm

Commit message: Final version without panelization.
Parts:
- added G***: LOGO, NadSilk:brain_logo_smol, F.Cu at (126.2, 138.3)
- added G***: LOGO, NadSilk:brain_logo, F.Cu at (123.4, 81.1)
- C11, C13, C14, C15, C16, C18, C19, C20, C21, C8, C9, D1, LS1, R12, R14, R15, R16, R19, R29, SW6, SW7, SW8, U12, U8: moved to B.Cu
- U10: value DD05CVSA -> DD04CVSA; footprint Retro_clock:DD05CVSA -> Retro_clock:DD04CVSA
- moved F1 220.7 mm to (73.5, 138.2), turned to 180 degrees
- moved LS1 197.4 mm to (122.4, 165.2), turned to -150 degrees
- moved R22 188.8 mm to (74.0, 148.2), turned to 90 degrees
- moved C16 181.9 mm to (80.1, 128.9), turned to 180 degrees
- moved C18 169.0 mm to (69.4, 134.0), turned to 180 degrees
- moved C19 167.2 mm to (73.2, 135.5)
- moved R25 159.6 mm to (69.3, 133.5), turned to -90 degrees
- moved C21 157.8 mm to (96.2, 158.2), turned to 180 degrees
- moved R26 156.5 mm to (71.4, 133.5), turned to -90 degrees
- moved C15 150.4 mm to (110.1, 184.9)
- moved C13 149.3 mm to (104.3, 185.5), turned to 180 degrees
- moved C14 147.4 mm to (110.8, 182.3)
- moved C17 145.2 mm to (77.7, 138.8), turned to -90 degrees
- moved R21 144.7 mm to (122.2, 194.7), turned to 90 degrees
- moved C20 143.1 mm to (99.9, 158.2)
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Connections:
- C6 pad 2: Net-(C6-Pad2) -> GND
- C7 pad 2: Net-(C6-Pad2) -> GND
- J3 pad 3: +3.3V -> +5V
- J3 pad 4: +5V -> +3.3V
- J4 pad 3: +3.3VP -> +5VP
- J4 pad 4: +5VP -> +3.3VP
- J7 pad 1: +3.3V -> +3.3VP
- R23 pad 1: +3.3V -> +3.3VP
- R24 pad 1: +3.3V -> +3.3VP
- U5 pad 10: N1_A -> N1_D
- U5 pad 11: N2_C -> N1_B
- U5 pad 12: N2_B -> N1_C
- U5 pad 2: Net-(C6-Pad2) -> +3.3VP
- U5 pad 26: ENC_CLK_ -> N2_A
- U5 pad 29: NX_SHDN -> N2_D
- U5 pad 31: SHIFT_DSA -> N2_B
- U5 pad 33: N1_C -> N2_C
- U5 pad 36: N1_B -> SHIFT_DSA
- U5 pad 37: N1_D -> ENC_CLK_
- U5 pad 8: N2_D -> NX_SHDN
- U5 pad 9: N2_A -> N1_A
Routing:
- net +3.3VP: track 0.00 -> 242.6 mm, vias 0 -> 3
- net GND: track 0.00 -> 197.7 mm, vias 0 -> 52
- net +5VP: track 0.00 -> 119.9 mm, vias 0 -> 6
- net NX_SHDN: track 0.00 -> 116.1 mm, vias 0 -> 2
- net N1_C: track 0.00 -> 107.4 mm, vias 0 -> 2
- net N2_C: track 0.00 -> 103.3 mm, vias 0 -> 2
- net N1_B: track 0.00 -> 103.0 mm, vias 0 -> 2
- net N1_D: track 0.00 -> 101.9 mm, vias 0 -> 2
- net N1_A: track 0.00 -> 100.5 mm, vias 0 -> 2
- net +12V: track 0.00 -> 94.7 mm
- net N2_B: track 0.00 -> 94.1 mm, vias 0 -> 2
- net BUTTON_Y: track 0.00 -> 93.0 mm, vias 0 -> 1
- net BUTTON_N: track 0.00 -> 88.2 mm, vias 0 -> 1
- net N2_D: track 0.00 -> 86.7 mm
- net ENC_DATA_: track 0.00 -> 85.2 mm, vias 0 -> 3
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Other:
- outline, holes or cut-outs redrawn

Commit message: Fixed some minor things, added panelization.
Parts:
- removed the G*** at (126.2, 138.3)
- added G***: LOGO, NadSilk:brain_logo, F.Cu at (229.2, 47.2)
- added mouse-bite-1mm-slot: VAL**, Panelization:mouse-bite-1mm-slot, F.Cu at (149.5, 92.0)
- added mouse-bite-1mm-slot: VAL**, Panelization:mouse-bite-1mm-slot, F.Cu at (149.5, 76.1)
- moved C13 135.0 mm to (205.1, 95.6)
- moved J5 134.9 mm to (194.5, 91.7)
- moved H5 134.7 mm to (154.0, 40.1)
- moved H6 134.7 mm to (154.0, 109.9)
- moved H7 134.7 mm to (286.6, 109.9)
- moved H8 134.7 mm to (286.6, 40.1)
- moved LS1 134.7 mm to (222.9, 75.6)
- moved R18 134.7 mm to (219.9, 106.0)
- moved R19 134.7 mm to (224.8, 103.2)
- moved R20 134.7 mm to (219.2, 103.9)
- moved U8 134.7 mm to (210.4, 100.1)
- moved BT1 134.7 mm to (242.0, 47.8)
- moved C10 134.7 mm to (240.0, 77.1)
- moved C14 134.7 mm to (211.3, 92.7)
- moved C15 134.7 mm to (210.6, 95.3)
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Routing:
- net GND: track 197.7 -> 212.9 mm, vias 52 -> 55
- net +5VP: track 119.9 -> 125.3 mm
- net VBUS: track 46.3 -> 45.8 mm
Other:
- board size 143.3 x 164.2 mm -> 280.9 x 76.8 mm
- board text added: "BOOT"
- board text added: "RST"
- board text added: "Volume down"
- board text added: "Volume up"
